File: RPi_Student/RPi_Student.kicad_sch (KiCad schematic)
At the start: 12 parts, among them J1 Conn_01x02, J2 Conn_01x02, J3 Conn_01x03, J4 GPIO, J5 Conn_01x06, J6 Conn_01x04, J7 Conn_01x02_Male, Q1 BC856BDW1, Q2 IRF9540N, U1 LM1085-ADJ

Commit message: Updated to account for new PCB design changes
Parts:
- added C1, C2: 10u, Capacitor_THT:CP_Radial_D5.0mm_P2.50mm, symbol Device:C_Polarized_US
- added C3, C4: 100u, Capacitor_Tantalum_SMD:CP_EIA-2012-12_Kemet-R_Pad1.30x1.05mm_HandSolder, symbol Device:C_Polarized_US
- added D1, D2: LED, Diode_SMD:D_0805_2012Metric_Pad1.15x1.40mm_HandSolder, symbol Device:LED
- added F1: MCCQ-122, RPi_Hat:MCCQ122, symbol MCQQ:MCCQ-122
- added Q3: IRF9540N, Package_TO_SOT_THT:TO-220-3_Vertical, symbol Transistor_FET:IRF9540N
- added R3, R5: 121, Resistor_SMD:R_0805_2012Metric_Pad1.20x1.40mm_HandSolder, symbol Device:R
- added R4, R6: 365, Resistor_SMD:R_0805_2012Metric_Pad1.20x1.40mm_HandSolder, symbol Device:R
- added R7, R8: R, Resistor_SMD:R_0805_2012Metric_Pad1.20x1.40mm_HandSolder, symbol Device:R
- added SW1, SW2: SW_SPDT, RPi_Hat:Switch_SPDT_Jaycar, symbol Switch:SW_SPDT
- added U2: LM1085-ADJ, RPi_Hat:LM1085-5.0, symbol Regulator_Linear:LM1085-ADJ
- J2: footprint Connector_PinSocket_2.54mm:PinSocket_1x02_P2.54mm_Vertical -> RPi_Hat:TE_282836-2
Connections:
- net 5v is gone; now on net +5V: J4.4 (Pin_4)
- net VDDF is gone; now on net VD: Q1.4 (E2), Q2.3 (S)
- net +5V: no longer J5.4 (Pin_4)
- net +BATT: now also D1.2 (A), SW2.1 (A)
- net GND: now also J7.1 (Pin_1), C1.2, C2.2, C3.2, C4.2, Q3.1 (G), R4.2, R6.2, R7.1, R8.2
- net VCC: now also U1.3 (VI), C1.1, C2.1, SW1.1 (A), U2.3 (VI)
- net VD: now also D2.2 (A)
- net VDDA: now also U1.2 (VO), C3.1, R3.1
- net Vdrive: now also C4.1, R5.1, U2.2 (VO)
- net at U1.1 (ADJ): now also R3.2, R4.1
- net at J7.2 (Pin_2): now also F1.1, F1.2
- new net: Q3.3 (S), SW1.2 (B), SW2.2 (B)
- new net: F1.3, F1.4, Q3.2 (D)
- new net: D2.1 (K), R8.1
- new net: D1.1 (K), R7.2
- new net: R5.2, R6.1, U2.1 (ADJ)
- no-connect marks 0 -> 3

Commit message: New layout for students to solve
Parts:
- removed C1, C2: 10u, Capacitor_THT:CP_Radial_D5.0mm_P2.50mm, symbol Device:C_Polarized_US
- removed C3, C4: 100u, Capacitor_Tantalum_SMD:CP_EIA-2012-12_Kemet-R_Pad1.30x1.05mm_HandSolder, symbol Device:C_Polarized_US
- removed R3, R5: 121, Resistor_SMD:R_0805_2012Metric_Pad1.20x1.40mm_HandSolder, symbol Device:R
- removed R4, R6: 365, Resistor_SMD:R_0805_2012Metric_Pad1.20x1.40mm_HandSolder, symbol Device:R
- removed R7, R8: R, Resistor_SMD:R_0805_2012Metric_Pad1.20x1.40mm_HandSolder, symbol Device:R
Connections:
- net +BATT: no longer D1.2 (A)
- net GND: no longer Q3.1 (G)
- net VCC: no longer U1.3 (VI), U2.3 (VI)
- net VD: no longer D2.2 (A)
- net VDDA: no longer U1.2 (VO)
- net Vdrive: no longer U2.2 (VO)
- net at SW1.2 (B), SW2.2 (B): no longer Q3.3 (S)
- now unconnected: F1.1, F1.2, F1.3, F1.4, J7.2 (Pin_2), Q3.2 (D)
Other:
- moved on the sheet: D1, D2, Q3, U1
